Commit message: Quase pronto

File: robot_description/urdf/robot.gazebo.xacro (robot description, xacro)
@@ -37,7 +37,7 @@
         <rightJoint>joint_right_wheel</rightJoint>
         <!-- The distance from the center of one wheel to the other, in meters, defaults to 0.34 m -->
-        <wheelSeparation>0.299998</wheelSeparation>
+        <wheelSeparation>0.407</wheelSeparation>
         <!-- Diameter of the wheels, in meters, defaults to 0.15 m -->
-        <wheelDiameter>0.10</wheelDiameter>
+        <wheelDiameter>0.1016</wheelDiameter>
         <!-- Wheel acceleration, in rad/s^2, defaults to 0.0 rad/s^2 -->
         <wheelAcceleration>0</wheelAcceleration>
@@ -74,5 +74,4 @@
         </plugin>
     </gazebo>
-        <!-- camera -->
     <gazebo reference="camera_1">
         <sensor type="camera" name="camera1">
@@ -92,7 +91,4 @@
                 <noise>
                 <type>gaussian</type>
-                <!-- Noise is sampled independently per pixel on each frame.
-                    That pixel's noise value is added to each of its color
-                    channels, which at that point lie in the range [0,1]. -->
                 <mean>0.0</mean>
                 <stddev>0.007</stddev>
@@ -115,3 +111,38 @@
         </sensor>
     </gazebo>
+  <gazebo reference="lidar">
+    <sensor type="ray" name="laser_sensor">
+      <pose>0 0 0 0 0 0</pose>
+      <visualize>false</visualize>
+      <update_rate>40</update_rate>
+      <ray>
+        <scan>
+          <horizontal>
+            <samples>720</samples>
+            <resolution>1</resolution>
+            <min_angle>-1.1775</min_angle>
+            <max_angle>1.1775</max_angle>
+          </horizontal>
+        </scan>
+        <range>
+          <min>0.10</min>
+          <max>10.0</max>
+          <resolution>0.01</resolution>
+        </range>
+        <noise>
+          <type>gaussian</type>
+          <!-- Noise parameters based on published spec for Hokuyo laser
+               achieving "+-30mm" accuracy at range < 10m.  A mean of 0.0m and
+               stddev of 0.01m will put 99.7% of samples within 0.03m of the true
+               reading. -->
+          <mean>0.0</mean>
+          <stddev>0.01</stddev>
+        </noise>
+      </ray>
+      <plugin name="gazebo_ros_head_hokuyo_controller" filename="libgazebo_ros_laser.so">
+        <topicName>/my_robot/laser/scan</topicName>
+        <frameName>lidar</frameName>
+      </plugin>
+    </sensor>
+  </gazebo>
 </robot>

File: robot_description/urdf/robot.urdf.xacro (robot description, xacro)
@@ -5,18 +5,43 @@
     <parent link="carcaca"/>
     <child link="camera_1"/>
-    <origin rpy="0 1.57 0" xyz="0 0.036515 0.03"/>
+    <origin rpy="0 1.57 0" xyz="0 -0.127 0.0367"/>
+  </joint>
+  <joint name="joint_lidar" type="fixed">
+    <parent link="carcaca"/>
+    <child link="lidar"/>
+    <origin rpy="0 0 -1.57" xyz="-0.0005 -0.23 0.109"/>
   </joint>
   <joint name="joint_lifting_tray" type="prismatic">
     <parent link="carcaca"/>
     <child link="lifting_tray"/>
-    <origin rpy="0 0 0" xyz="0 0.07 0.108"/>
+    <origin rpy="0 0 0" xyz="0 0 0.1318"/>
     <axis xyz="0 0 1"/>
-    <limit effort="10" lower="0" upper="0.10" velocity="0.05"/>
+    <limit effort="100" lower="0" upper="0.04" velocity="1"/>
+  </joint>
+  <joint name="joint_wheel_front_right" type="fixed">
+    <parent link="carcaca"/>
+    <child link="wheel_front_right"/>
+    <origin rpy="0 1.57 0" xyz="0.193 -0.176 0.0508"/>
+  </joint>
+  <joint name="joint_wheel_rear_right" type="fixed">
+    <parent link="carcaca"/>
+    <child link="wheel_rear_right"/>
+    <origin rpy="0 1.57 0" xyz="0.193 0.176 0.0508"/>
+  </joint>
+  <joint name="joint_wheel_front_left" type="fixed">
+    <parent link="carcaca"/>
+    <child link="wheel_front_left"/>
+    <origin rpy="0 1.57 0" xyz="-0.214 -0.176 0.0508"/>
+  </joint>
+  <joint name="joint_wheel_rear_left" type="fixed">
+    <parent link="carcaca"/>
+    <child link="wheel_rear_left"/>
+    <origin rpy="0 1.57 0" xyz="-0.214 0.176 0.0508"/>
   </joint>
   <joint name="joint_right_wheel" type="revolute">
     <parent link="carcaca"/>
     <child link="right_wheel"/>
-    <origin rpy="0     -1.5707  0" xyz="0.19   0.036515  0.04645"/>
-    <axis xyz="0   0   -1"/>
+    <origin rpy="0 1.57 0" xyz="0.193 0 0.0507"/>
+    <axis xyz="0 0 1"/>
     <limit effort="-1.0" lower="-1e+16" upper="1e+16" velocity="-1.0"/>
   </joint>
@@ -24,24 +49,24 @@
     <parent link="carcaca"/>
     <child link="left_wheel"/>
-    <origin rpy="0      1.5707  0" xyz="-0.19   0.036515  0.04645"/>
-    <axis xyz="0   0   1"/>
+    <origin rpy="0 1.57 0" xyz="-0.214 0 0.0507"/>
+    <axis xyz="0 0 1"/>
     <limit effort="-1.0" lower="-1e+16" upper="1e+16" velocity="-1.0"/>
   </joint>
   <gazebo reference="carcaca">
     <selfCollide>true</selfCollide>
-    <mu1 value="0.05"/>
-    <mu2 value="0.05"/>
-    <kp value="10000000.0" />
-    <kd value="1" />
+    <mu1 value="0.3"/>
+    <mu2 value="0.3"/>
+    <kp value="10000000.0" />
+    <kd value="1000" />
     <fdir1 value="0 0 0"/>
   </gazebo>
   <link name="carcaca">
     <inertial>
-      <mass value="20"/>
-      <origin rpy="0  0  3.14" xyz="0  0  0"/>
+      <mass value="15"/>
+      <origin rpy="0  0  3.14" xyz="0  0  0.0118"/>
       <inertia ixx="1" ixy="0" ixz="0" iyy="1" iyz="0" izz="1"/>
     </inertial>
     <collision name="carcaca_collision">
-      <origin rpy="0  0  3.14" xyz="0  0  0"/>
+      <origin rpy="0  0  3.14" xyz="0  0  0.0118"/>
       <geometry>
         <mesh filename="package://robot_description/models/laser_robot/meshes/carcaca.dae" scale="1 1 1"/>
@@ -49,7 +74,115 @@
     </collision>
     <visual name="carcaca_visual">
-      <origin rpy="0  0  3.14" xyz="0  0  0"/>
-      <geometry>
-        <mesh filename="package://robot_description/models/laser_robot/meshes/carcaca.dae" scale="1.0 1.0 1.0"/>
+      <origin rpy="0  0  3.14" xyz="0  0  0.0118"/>
+      <geometry>
+        <mesh filename="package://robot_description/models/laser_robot/meshes/carcaca.dae" scale="1 1 1"/>
+      </geometry>
+    </visual>
+  </link>
+  <gazebo reference="wheel_front_right">
+    <selfCollide>true</selfCollide>
+    <mu1 value="0.09"/>
+    <mu2 value="0.09"/>
+    <kp value="10000000.0" />
+    <kd value="10000" />
+    <fdir1 value="0 0 0"/>
+  </gazebo>
+  <link name="wheel_front_right">
+    <inertial>
+      <mass value="0.01"/>
+      <origin rpy="0 0 0" xyz="0 0 0"/>
+      <inertia ixx="1" ixy="0.0" ixz="0.0" iyy="1" iyz="0.0" izz="1"/>
+    </inertial>
+    <collision name="wheel_front_right_collision">
+      <origin rpy="0 0 0" xyz="0 0 0"/>
+      <geometry>
+        <mesh filename="package://robot_description/models/laser_robot/omni_wheel/meshes/roda_omni.obj" scale="1 1 1"/>
+      </geometry>
+    </collision>
+    <visual name="wheel_front_right_visual">
+      <origin rpy="0 0 0" xyz="0 0 0"/>
+      <geometry>
+        <mesh filename="package://robot_description/models/laser_robot/omni_wheel/meshes/roda_omni.obj" scale="1 1 1"/>
+      </geometry>
+    </visual>
+  </link>
+  <gazebo reference="wheel_rear_right">
+    <selfCollide>true</selfCollide>
+    <mu1 value="0.09"/>
+    <mu2 value="0.09"/>
+    <kp value="10000000.0" />
+    <kd value="10000" />
+    <fdir1 value="0 0 0"/>
+  </gazebo>
+  <link name="wheel_rear_right">
+    <inertial>
+      <mass value="0.01"/>
+      <origin rpy="0 0 0" xyz="0 0 0"/>
+      <inertia ixx="1" ixy="0.0" ixz="0.0" iyy="1" iyz="0.0" izz="1"/>
+    </inertial>
+    <collision name="wheel_rear_right_collision">
+      <origin rpy="0 0 0" xyz="0 0 0"/>
+      <geometry>
+        <mesh filename="package://robot_description/models/laser_robot/omni_wheel/meshes/roda_omni.obj" scale="1 1 1"/>
+      </geometry>
+    </collision>
+    <visual name="wheel_rear_right_visual">
+      <origin rpy="0 0 0" xyz="0 0 0"/>
+      <geometry>
+        <mesh filename="package://robot_description/models/laser_robot/omni_wheel/meshes/roda_omni.obj" scale="1 1 1"/>
+      </geometry>
+    </visual>
+  </link>
+  <gazebo reference="wheel_front_left">
+    <selfCollide>true</selfCollide>
+    <mu1 value="0.09"/>
+    <mu2 value="0.09"/>
+    <kp value="10000000.0" />
+    <kd value="10000" />
+    <fdir1 value="0 0 0"/>
+  </gazebo>
+  <link name="wheel_front_left">
+    <inertial>
+      <mass value="0.01"/>
+      <origin rpy="0 0 0" xyz="0 0 0"/>
+      <inertia ixx="1" ixy="0.0" ixz="0.0" iyy="1" iyz="0.0" izz="1"/>
+    </inertial>
+    <collision name="wheel_front_left_collision">
+      <origin rpy="0 0 0" xyz="0 0 0"/>
+      <geometry>
+        <mesh filename="package://robot_description/models/laser_robot/omni_wheel/meshes/roda_omni.obj" scale="1 1 1"/>
+      </geometry>
+    </collision>
+    <visual name="wheel_front_left_visual">
+      <origin rpy="0 0 0" xyz="0 0 0"/>
+      <geometry>
+        <mesh filename="package://robot_description/models/laser_robot/omni_wheel/meshes/roda_omni.obj" scale="1 1 1"/>
+      </geometry>
+    </visual>
+  </link>
+  <gazebo reference="wheel_rear_left">
+    <selfCollide>true</selfCollide>
+    <mu1 value="0.09"/>
+    <mu2 value="0.09"/>
+    <kp value="10000000.0" />
+    <kd value="10000" />
+    <fdir1 value="0 0 0"/>
+  </gazebo>
+  <link name="wheel_rear_left">
+    <inertial>
+      <mass value="0.01"/>
+      <origin rpy="0 0 0" xyz="0 0 0"/>
+      <inertia ixx="1" ixy="0.0" ixz="0.0" iyy="1" iyz="0.0" izz="1"/>
+    </inertial>
+    <collision name="wheel_rear_left_collision">
+      <origin rpy="0 0 0" xyz="0 0 0"/>
+      <geometry>
+        <mesh filename="package://robot_description/models/laser_robot/omni_wheel/meshes/roda_omni.obj" scale="1 1 1"/>
+      </geometry>
+    </collision>
+    <visual name="wheel_rear_left_visual">
+      <origin rpy="0 0 0" xyz="0 0 0"/>
+      <geometry>
+        <mesh filename="package://robot_description/models/laser_robot/omni_wheel/meshes/roda_omni.obj" scale="1 1 1"/>
       </geometry>
     </visual>
@@ -57,6 +190,6 @@
   <gazebo reference="lifting_tray">
     <selfCollide>true</selfCollide>
-    <mu1 value="100"/>
-    <mu2 value="50"/>
+    <mu1 value="0.1"/>
+    <mu2 value="0.1"/>
     <kp value="10000000.0" />
     <kd value="10000" />
@@ -66,17 +199,17 @@
     <inertial>
       <mass value="0.5"/>
-      <origin rpy="0  0  0" xyz="0  0 0"/>
+      <origin rpy="0  0  0" xyz="0 0 0"/>
       <inertia ixx="1" ixy="0" ixz="0" iyy="1" iyz="0" izz="1"/>
     </inertial>
     <collision name="lifting_tray_collision">
-      <origin rpy="0  0  0" xyz="0 0 -0.108"/>
-      <geometry>
-        <mesh filename="package://robot_description/models/laser_robot/meshes/pistao.dae" scale="1 1 1"/>
+      <origin rpy="0  0  0" xyz="0 0 0"/>
+      <geometry>
+        <mesh filename="package://robot_description/models/laser_robot/meshes/lifting.dae" scale="1 1 1"/>
       </geometry>
     </collision>
     <visual name="lifting_tray_visual">
-      <origin rpy="0  0  0" xyz="0 0 -0.108"/>
-      <geometry>
-        <mesh filename="package://robot_description/models/laser_robot/meshes/pistao.dae" scale="1.0 1.0 1.0"/>
+      <origin rpy="0  0  0" xyz="0 0 0"/>
+      <geometry>
+        <mesh filename="package://robot_description/models/laser_robot/meshes/lifting.dae" scale="1 1 1"/>
       </geometry>
     </visual>
@@ -85,17 +218,17 @@
     <inertial>
       <mass value="0.1"/>
-      <origin rpy="0 1.57 0" xyz="0 0 0.01"/>
+      <origin rpy="0 0 0" xyz="0 0 0"/>
       <inertia ixx="1" ixy="0" ixz="0" iyy="1" iyz="0" izz="1"/>
     </inertial>
     <collision name="camera_1_collision">
-      <origin rpy="0 1.57 0" xyz="0 0 0"/>
-      <geometry>
-        <mesh filename="package://robot_description/models/laser_robot/meshes/camera_1.dae" scale="1 1 1"/>
+      <origin rpy="0 0 0" xyz="0 0 0"/>
+      <geometry>
+        <mesh filename="package://robot_description/models/laser_robot/camera/meshes/camera.obj" scale="0.5 0.5 0.5"/>
       </geometry>
     </collision>
     <visual name="camera_1_visual">
-      <origin rpy="0 1.57 0" xyz="0 0 0"/>
-      <geometry>
-        <mesh filename="package://robot_description/models/laser_robot/meshes/camera_1.dae" scale="1.0 1.0 1.0"/>
+      <origin rpy="0 0 1.57" xyz="0 0 0"/>
+      <geometry>
+        <mesh filename="package://robot_description/models/laser_robot/camera/meshes/camera.obj" scale="0.5 0.5 0.5"/>
       </geometry>
     </visual>
@@ -106,11 +239,11 @@
     <mu2 value="50"/>
     <kp value="10000000.0" />
-    <kd value="1" />
-    <fdir1 value="1 0 0"/>
+    <kd value="1000" />
+    <fdir1 value="0 0 0"/>
   </gazebo>
   <link name="right_wheel">
     <inertial>
       <mass value="1"/>
-      <origin rpy="0  0  0" xyz="0  0  0"/>
+      <origin rpy="0 0 0" xyz="0 0 0"/>
       <inertia ixx="1" ixy="0" ixz="0" iyy="1" iyz="0" izz="1"/>
     </inertial>
@@ -118,5 +251,5 @@
       <origin rpy="0 0 0" xyz="0 0 0"/>
       <geometry>
-        <mesh filename="package://robot_description/models/laser_robot/meshes/roda.dae" scale="1 1 1"/>
+        <mesh filename="package://robot_description/models/laser_robot/wheel/meshes/roda.obj" scale="1 1 1"/>
       </geometry>
     </collision>
@@ -124,5 +257,5 @@
       <origin rpy="0 0 0" xyz="0 0 0"/>
       <geometry>
-        <mesh filename="package://robot_description/models/laser_robot/meshes/roda.dae" scale="1.0 1.0 1.0"/>
+        <mesh filename="package://robot_description/models/laser_robot/wheel/meshes/roda.obj" scale="1 1 1"/>
       </geometry>
     </visual>
@@ -133,6 +266,6 @@
     <mu2 value="50"/>
     <kp value="10000000.0" />
-    <kd value="1" />
-    <fdir1 value="1 0 0"/>
+    <kd value="1000" />
+    <fdir1 value="0 0 0"/>
   </gazebo>
   <link name="left_wheel">
@@ -145,5 +278,5 @@
       <origin rpy="0 0 0" xyz="0 0 0"/>
       <geometry>
-        <mesh filename="package://robot_description/models/laser_robot/meshes/roda.dae" scale="1 1 1"/>
+        <mesh filename="package://robot_description/models/laser_robot/wheel/meshes/roda.obj" scale="1 1 1"/>
       </geometry>
     </collision>
@@ -151,5 +284,24 @@
       <origin rpy="0 0 0" xyz="0 0 0"/>
       <geometry>
-        <mesh filename="package://robot_description/models/laser_robot/meshes/roda.dae" scale="1.0 1.0 1.0"/>
+        <mesh filename="package://robot_description/models/laser_robot/wheel/meshes/roda.obj" scale="1 1 1"/>
+      </geometry>
+    </visual>
+  </link>
+  <link name="lidar">
+    <inertial>
+      <mass value="0.1"/>
+      <origin rpy="0 0 0" xyz="0 0 0"/>
+      <inertia ixx="1" ixy="0" ixz="0" iyy="1" iyz="0" izz="1"/>
+    </inertial>
+    <collision name="lidar_collision">
+      <origin rpy="0 0 0" xyz="0 0 0"/>
+      <geometry>
+        <mesh filename="package://robot_description/models/laser_robot/lidar/meshes/lidar.obj" scale="0.5 0.5 0.5"/>
+      </geometry>
+    </collision>
+    <visual name="lidar_visual">
+      <origin rpy="0 1.57 1.57" xyz="0 0 0"/>
+      <geometry>
+        <mesh filename="package://robot_description/models/laser_robot/lidar/meshes/lidar.obj" scale="0.5 0.5 0.5"/>
       </geometry>
     </visual>
